Commit message: 添加新的load_gym.py文件，初始化Isaac Gym模拟环境，创建足球场、机器人和足球的URDF资源，并设置相机和物理参数以支持仿真。

File: booster_gym-main/resources/T1/soccer_field_half.urdf (robot description, URDF)
Before this commit: robot soccer_field_half, 22 links, 21 joints
Links:
- link crossbar: mass None -> 10.0
- link field_base: mass None -> 1000.0
- link left_goal_post: mass None -> 10.0
- link right_goal_post: mass None -> 10.0
