Commit message: 优化足球场半场URDF文件，合并场地线条为一个链接以减少渲染开销，调整多个链接的高度和质量参数，提升整体视觉效果和物理表现。

File: booster_gym-main/resources/T1/soccer_ball_optimized.urdf (robot description, URDF)
Before this commit: robot soccer_ball, 1 links, 0 joints
Links:
- link soccer_ball: geometry collision sphere radius=0.11; visual cylinder length=0.12 radius=0.005

File: booster_gym-main/resources/T1/soccer_field_half.urdf (robot description, URDF)
Before this commit: robot soccer_field_half, 22 links, 21 joints
Links:
- removed link back_crossbar
- removed link center_circle_arc_1
- removed link center_circle_arc_2
- removed link center_circle_arc_3
- removed link crossbar
- removed link goal_line
- removed link left_corner_arc_1
- removed link left_corner_arc_2
- removed link left_goal_back
- removed link left_goal_post
- removed link left_touchline
- removed link midfield_line
- removed link penalty_area_front
- removed link penalty_area_left
- removed link penalty_area_right
- removed link penalty_spot
- removed link right_corner_arc_1
- removed link right_corner_arc_2
- removed link right_goal_back
- removed link right_goal_post
- removed link right_touchline
- added link field_lines; visual box size=0.1 2.2 0.001; visual box size=0.1 2.2 0.001
- added link goal_structure, mass 50.0; collision cylinder length=0.8 radius=0.05; collision cylinder length=0.8 radius=0.05
- link field_base: geometry collision box size=12 9 0.01; visual box size=12 9 0.01
Joints:
- removed joint field_to_back_crossbar
- removed joint field_to_center_circle_arc_1
- removed joint field_to_center_circle_arc_2
- removed joint field_to_center_circle_arc_3
- removed joint field_to_crossbar
- removed joint field_to_goal_line
- removed joint field_to_left_corner_arc_1
- removed joint field_to_left_corner_arc_2
- removed joint field_to_left_goal_back
- removed joint field_to_left_goal_post
- removed joint field_to_left_touchline
- removed joint field_to_midfield_line
- removed joint field_to_penalty_area_front
- removed joint field_to_penalty_area_left
- removed joint field_to_penalty_area_right
- removed joint field_to_penalty_spot
- removed joint field_to_right_corner_arc_1
- removed joint field_to_right_corner_arc_2
- removed joint field_to_right_goal_back
- removed joint field_to_right_goal_post
- removed joint field_to_right_touchline
- added joint field_to_goal: type fixed, parent field_base, child goal_structure
- added joint field_to_lines: type fixed, parent field_base, child field_lines
